Commit message: updates for t265

File: realsense2_description/urdf/_t265.urdf.xacro (robot description, xacro)
@@ -8,5 +8,5 @@
 <robot name="sensor_t265" xmlns:xacro="http://ros.org/wiki/xacro">
   <!--File includes-->
-  <xacro:include filename="$(find realsense_simulation)/urdf/_t265.gazebo.xacro"/>
+  <xacro:include filename="$(find realsense2_description)/urdf/_materials.urdf.xacro" />
   <xacro:macro name="sensor_t265" params="parent name:=camera topics_ns:=camera *origin">
     <xacro:property name="M_PI" value="3.1415926535897931" />
@@ -19,7 +19,4 @@
     <xacro:property name="fisheye2_offset_y" value="0.0"/>
     <xacro:property name="fisheye2_offset_z" value="0.0"/>
-    <material name="${name}_aluminum">
-      <color rgba="0.5 0.5 0.5 1"/>
-    </material>
     <!-- camera body, with origin at camera_link -->
     <joint name="${name}_pose_frame_joint" type="fixed">
@@ -30,5 +27,5 @@
     <link name="${name}_pose_frame"/>
     <joint name="${name}_pose_joint" type="fixed">
-      <origin xyz="0 0 0" rpy="${90 * deg_to_rad} 0 ${-90 * deg_to_rad}"/>
+      <origin xyz="0 0 0" rpy="${M_PI/2} 0 ${M_PI/2}"/>
       <parent link="${name}_pose_frame"/>
       <child link="${name}_link" />
@@ -40,5 +37,5 @@
             <mesh filename="package://realsense2_description/meshes/t265.stl" />
         </geometry>
-        <material name="${name}_aluminum"/>
+        <material name="aluminum"/>
       </visual>
       <collision>
@@ -92,6 +89,4 @@
     </joint>
     <link name="${name}_accel_optical_frame"/>
-    <!-- Realsense Gazebo Plugin -->
-    <xacro:gazebo_t265 camera_name="${name}" fisheye1_reference_link="${name}_fisheye1_rgb_frame" fisheye2_reference_link="${name}_fisheye2_rgb_frame" topics_ns="${topics_ns}" fisheye1_optical_frame="${name}_fisheye1_optical_frame" fisheye2_optical_frame="${name}_fisheye2_optical_frame"/>
   </xacro:macro>
 </robot>

File: realsense2_description/urdf/test_t265_camera.urdf.xacro (robot description, xacro)
@@ -3,6 +3,6 @@
   <xacro:include filename="$(find realsense2_description)/urdf/_t265.urdf.xacro" />
   <link name="base_link" />
-  <sensor_t265 parent="base_link">
+  <xacro:sensor_t265 parent="base_link">
     <origin xyz="0 0 0" rpy="0 0 0"/>
-  </sensor_t265>
+  </xacro:sensor_t265>
 </robot>

Commit message: fixes for tfs

File: realsense2_description/urdf/_t265.urdf.xacro (robot description, xacro)
@@ -13,9 +13,9 @@
     <!-- The following values are approximate, and the camera node
      publishing TF values with actual calibrated camera extrinsic values -->
-    <xacro:property name="fisheye1_offset_x" value="-0.0411"/>
-    <xacro:property name="fisheye1_offset_y" value="0.0"/>
+    <xacro:property name="fisheye1_offset_y" value="0.0411"/>
+    <xacro:property name="fisheye1_offset_x" value="0.0"/>
     <xacro:property name="fisheye1_offset_z" value="0.0"/>
-    <xacro:property name="fisheye2_offset_x" value="0.0229"/>
-    <xacro:property name="fisheye2_offset_y" value="0.0"/>
+    <xacro:property name="fisheye2_offset_y" value="-0.0229"/>
+    <xacro:property name="fisheye2_offset_x" value="0.0"/>
     <xacro:property name="fisheye2_offset_z" value="0.0"/>
     <!-- camera body, with origin at camera_link -->
@@ -27,5 +27,5 @@
     <link name="${name}_pose_frame"/>
     <joint name="${name}_pose_joint" type="fixed">
-      <origin xyz="0 0 0" rpy="${M_PI/2} 0 ${M_PI/2}"/>
+      <origin xyz="0 0 0" rpy="0 ${M_PI/2} ${M_PI/2}"/>
       <parent link="${name}_pose_frame"/>
       <child link="${name}_link" />
@@ -33,5 +33,5 @@
     <link name="${name}_link">
       <visual>
-      <origin xyz="0 0 0" rpy="0 0 0"/>
+      <origin xyz="0 0 0" rpy="${M_PI/2} 0 -${M_PI/2}"/>
         <geometry>
             <mesh filename="package://realsense2_description/meshes/t265.stl" />
@@ -40,5 +40,5 @@
       </visual>
       <collision>
-        <origin xyz="0 0 0" rpy="0 0 0"/>
+        <origin xyz="0 0 0" rpy="${M_PI/2} 0 -${M_PI/2}"/>
         <geometry>
           <mesh filename="package://realsense2_description/meshes/t265.stl" />
@@ -53,5 +53,5 @@
     </link>
     <joint name="${name}_fisheye1_rgb_joint" type="fixed">
-      <origin xyz="${fisheye1_offset_x} ${fisheye1_offset_y} ${fisheye1_offset_z}" rpy="0 ${M_PI/2} ${M_PI/2}"/>
+      <origin xyz="${fisheye1_offset_x} ${fisheye1_offset_y} ${fisheye1_offset_z}" rpy="0 0 0"/>
       <parent link="${name}_link"/>
       <child link="${name}_fisheye1_rgb_frame" />
@@ -59,5 +59,5 @@
     <link name="${name}_fisheye1_rgb_frame"/>
     <joint name="${name}_fisheye2_rgb_joint" type="fixed">
-      <origin xyz="${fisheye2_offset_x} ${fisheye2_offset_y} ${fisheye2_offset_z}" rpy="0 ${M_PI/2} ${M_PI/2}"/>
+      <origin xyz="${fisheye2_offset_x} ${fisheye2_offset_y} ${fisheye2_offset_z}" rpy="0 0 0"/>
       <parent link="${name}_link"/>
       <child link="${name}_fisheye2_rgb_frame" />
@@ -78,5 +78,5 @@
     <!-- camera depth joints and links -->
     <joint name="${name}_gyro_optical_joint" type="fixed">
-      <origin xyz="-0.0311 0 0.00655" rpy="0 ${M_PI} 0"/>
+      <origin xyz="-0.00655 0.0311 0" rpy="${M_PI/2} 0 ${M_PI/2}"/>
       <parent link="${name}_link"/>
       <child link="${name}_gyro_optical_frame" />
